File: E15.kicad_pcb (KiCad board)
At the start: 2 copper layers, 48.4 x 21.6 mm, 26 parts, among them J1 2x2 Connector, J2 WS-bus output, J3 WS-bus input, J4 UPDI, J5 Debug, J7 Screw Connector, U1 AVR-64da32, U2 MIC5205-5.0YM5

Commit message: Initial commit
Other:
- rule pad_to_mask_clearance: 0.051 -> 0
- board text added: "E15.1"
- board text removed: "E15.0"
Changed lines of the file:
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@@
     (company "Frank Schumacher")
     (comment 1 "WS2811 chip emulator for 12 multiplex LEDs (fixed voltage)")
+    (comment 4 "Licensed under the Apache License, Version 2")
   )
   (layers
@@
     (pad_size 1 0.5)
     (pad_drill 0)
-    (pad_to_mask_clearance 0.051)
-    (solder_mask_min_width 0.1)
+    (pad_to_mask_clearance 0)
     (aux_axis_origin 0 0)
     (visible_elements 7FFFFFFF)
@@
     (effects (font (size 1 1) (thickness 0.15)) (justify mirror))
   )
-  (gr_text E15.0 (at 101.49 89.04) (layer F.Cu)
+  (gr_text E15.1 (at 101.49 89.04) (layer F.Cu)
     (effects (font (size 1 1) (thickness 0.15)))
   )

Commit message: initial
Parts:
- D1: value SSL34F -> SSA33L; footprint Diode_SMD:D_SOD-123F -> Diode_SMD:D_SMA
- J1: value 2x2 Connector -> MPX output
- J4: value UPDI -> UPDI IF
- J5: value Debug -> Debug IF
- J7: value Screw Connector -> MPX output
- R20: moved to F.Cu
- moved R20 3.66 mm to (117.0, 95.7), turned to 180 degrees
- moved JP1 0.22 mm to (127.8, 81.6)
- moved U2 0.22 mm to (127.8, 78.4)
- moved D1 0.17 mm to (133.1, 87.6)
Routing:
- net GND: track 8.47 -> 20.0 mm, vias 8 -> 6
- net VDD: track 18.4 -> 15.0 mm, vias 2 -> 1
- net Net-(D2-Pad2): track 0.00 -> 2.09 mm, vias 1 -> 0
- net DI: track 7.62 -> 8.19 mm
