File: E15.kicad_pcb (KiCad board)
At the start: 2 copper layers, 48.4 x 21.6 mm, 26 parts, among them J1 MPX output, J2 WS-bus output, J3 WS-bus input, J4 UPDI IF, J5 Debug IF, J7 MPX output, U1 AVR-64da32, U2 MIC5205-5.0YM5

Commit message: mod: documentation
Routing:
- net GND: track 20.0 -> 15.7 mm
Changed lines of the file:
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@@
     (thickness 1.6)
     (drawings 27)
-    (tracks 181)
+    (tracks 176)
     (zones 0)
     (modules 26)
@@
   (title_block
     (title "RTB E15 module")
-    (date 2023-12-30)
+    (date 2024-11-14)
     (rev 1)
     (company "Frank Schumacher")
@@
   (via (at 121.7 90.43) (size 0.6) (drill 0.3) (layers F.Cu B.Cu) (net 1))
   (via (at 119.49 90.44) (size 0.6) (drill 0.3) (layers F.Cu B.Cu) (net 1))
-  (segment (start 135.925 89.165) (end 136.23 88.86) (width 0.5) (layer B.Cu) (net 1))
   (segment (start 114.89 90.17) (end 115.621992 90.901992) (width 0.25) (layer F.Cu) (net 1))
   (segment (start 119.55334 90.424) (end 120.614 90.424) (width 0.25) (layer F.Cu) (net 1))
@@
   (segment (start 127.79 76.64) (end 127.915001 76.514999) (width 0.15) (layer F.Cu) (net 1))
   (segment (start 127.79 77.32) (end 127.79 76.64) (width 0.15) (layer F.Cu) (net 1))
-  (segment (start 135.93 89.16) (end 136.23 88.86) (width 0.5) (layer F.Cu) (net 1))
-  (segment (start 135.93 88.95) (end 135.93 89.16) (width 0.5) (layer F.Cu) (net 1))
-  (segment (start 136.06 89.03) (end 136.23 88.86) (width 0.5) (layer B.Cu) (net 1))
-  (segment (start 133.096 89.03) (end 136.06 89.03) (width 0.5) (layer B.Cu) (net 1))
   (segment (start 136.125 86.215) (end 136.23 86.32) (width 0.5) (layer B.Cu) (net 2))
   (segment (start 126.915001 78.175001) (end 126.84 78.1) (width 0.25) (layer F.Cu) (net 2))
